Commit message: add moveit, gazebo simulation

File: xr_tank/robot_model/xr_tank_arm.urdf.xacro (robot description, xacro)
@@ -1,4 +1,8 @@
 <?xml version="1.0"?>
-<robot name="topower_v1" xmlns:xacro="http://www.ros.org/wiki/xacro">
+<robot name="xr_tank" xmlns:xacro="http://www.ros.org/wiki/xacro">
+    <xacro:property name="arm_base_x" value="0.03"/>
+    <xacro:property name="arm_base_y" value="0.06"/>
+    <xacro:property name="arm_base_z" value="0.01"/>
+    <xacro:property name="arm_base_mass" value="0.5"/>
     <xacro:property name="arm_a_x" value="0.03"/>
     <xacro:property name="arm_a_y" value="0.06"/>
@@ -21,4 +25,5 @@
     <xacro:property name="gripper_open_dist" value="0.03"/>
     <link name="arm_root" />
+    <xacro:box_link name="arm_base" size_x="${arm_base_x}" size_y="${arm_base_y}" size_z="${arm_base_z}" mass="${arm_base_mass}" material="black" ori="0 0 ${0.5*arm_base_z}" />
     <xacro:box_link name="arm_a" size_x="${arm_a_x}" size_y="${arm_a_y}" size_z="${arm_a_z}" mass="${arm_a_mass}" material="white" ori="0 0 ${0.5*arm_a_z}" />
     <xacro:box_link name="arm_b" size_x="${arm_b_x}" size_y="${arm_b_y}" size_z="${arm_b_z}" mass="${arm_b_mass}" material="grey" ori="0 0 ${0.5*arm_b_z}" />
@@ -26,9 +31,14 @@
     <xacro:box_link name="gripper_l" size_x="${gripper_x}" size_y="${gripper_y}" size_z="${gripper_z}" mass="${gripper_mass}" material="white" />
     <xacro:box_link name="gripper_r" size_x="${gripper_x}" size_y="${gripper_y}" size_z="${gripper_z}" mass="${gripper_mass}" material="grey" />
+    <joint name="joint_arm_base" type="fixed">
+        <parent link="arm_root"/>
+        <child link="arm_base"/>
+        <origin xyz="0 0 ${0.5*body_z}" rpy="0 0 0"/>
+    </joint>
     <joint name="joint_arm_a" type="revolute">
-        <parent link="arm_root"/>
+        <parent link="arm_base"/>
         <child link="arm_a"/>
         <axis xyz="0 1 0"/>
-        <origin xyz="0 0 ${0.5*body_z}" rpy="0 0 0"/>
+        <origin xyz="0 0 ${arm_base_z}" rpy="0 0 0"/>
         <limit lower="${-0.5*PI}" upper="${0.5*PI}" effort="12" velocity="0.9" />
     </joint>

File: xr_tank/robot_model/xr_tank_common.xacro (robot description, xacro)
@@ -1,4 +1,4 @@
 <?xml version="1.0"?>
-<robot name="topower_v1" xmlns:xacro="http://www.ros.org/wiki/xacro">
+<robot name="xr_tank" xmlns:xacro="http://www.ros.org/wiki/xacro">
     <xacro:property name="PI" value="3.1415926"/>
     <xacro:macro name="visualAsCollision" params="*origin *geometry *material">

File: xr_tank/robot_model/xr_tank_pan_tilt_cam.urdf.xacro (robot description, xacro)
@@ -1,4 +1,4 @@
 <?xml version="1.0"?>
-<robot name="topower_v1" xmlns:xacro="http://www.ros.org/wiki/xacro">
+<robot name="xr_tank" xmlns:xacro="http://www.ros.org/wiki/xacro">
     <xacro:property name="pan_base_x" value="0.06"/>
     <xacro:property name="pan_base_y" value="0.04"/>

File: xr_tank/robot_model/xr_tank_vehicle.urdf.xacro (robot description, xacro)
@@ -1,4 +1,4 @@
 <?xml version="1.0"?>
-<robot name="topower_v1" xmlns:xacro="http://www.ros.org/wiki/xacro">
+<robot name="xr_tank" xmlns:xacro="http://www.ros.org/wiki/xacro">
     <xacro:property name="body_x" value="0.3"/>
     <xacro:property name="body_y" value="0.15"/>
@@ -11,10 +11,9 @@
     <xacro:property name="track_x" value="0.3"/>
     <xacro:property name="track_y" value="0.04"/>
-    <xacro:property name="track_z" value="0.12"/>
+    <xacro:property name="track_z" value="0.10"/>
     <xacro:property name="track_mass" value="0.4"/>
     <xacro:property name="wheel_radius" value="0.06"/>
     <xacro:property name="wheel_height" value="0.05"/>
     <xacro:property name="wheel_mass" value="0.1"/>
-    <xacro:property name="wheel_offset_x" value="0.065"/>
     <xacro:property name="wheel_offset_z" value="-0.01"/>
     <!-- ==================body======================= -->
@@ -35,9 +34,11 @@
     <xacro:cylinder_link name="wheel_l" radius="${wheel_radius}" height="${wheel_height}" mass="${wheel_mass}" material="black"/>
     <xacro:cylinder_link name="wheel_r" radius="${wheel_radius}" height="${wheel_height}" mass="${wheel_mass}" material="black"/>
+    <xacro:cylinder_link name="passive_wheel_l" radius="${wheel_radius}" height="${wheel_height}" mass="${wheel_mass}" material="black"/>
+    <xacro:cylinder_link name="passive_wheel_r" radius="${wheel_radius}" height="${wheel_height}" mass="${wheel_mass}" material="black"/>
     <joint name="joint_wheel_l" type="continuous">
         <parent link="vehicle_body"/>
         <child link="wheel_l"/>
         <axis xyz="0 0 1"/>
-        <origin xyz="${-wheel_offset_x} ${0.5*(body_y+wheel_height)} ${wheel_offset_z}" rpy="${PI*0.5} 0 0"/>
+        <origin xyz="${-0.5*body_x+wheel_radius} ${0.5*(body_y+wheel_height)} ${wheel_offset_z}" rpy="${PI*0.5} 0 0"/>
     </joint>
     <joint name="joint_wheel_r" type="continuous">
@@ -45,5 +46,15 @@
         <child link="wheel_r"/>
         <axis xyz="0 0 1"/>
-        <origin xyz="${-wheel_offset_x} ${-0.5*(body_y+wheel_height)} ${wheel_offset_z}" rpy="${PI*0.5} 0 0"/>
+        <origin xyz="${-0.5*body_x+wheel_radius} ${-0.5*(body_y+wheel_height)} ${wheel_offset_z}" rpy="${PI*0.5} 0 0"/>
+    </joint>
+    <joint name="joint_passive_wheel_l" type="fixed">
+        <parent link="vehicle_body"/>
+        <child link="passive_wheel_l"/>
+        <origin xyz="${0.5*body_x-wheel_radius} ${0.5*(body_y+wheel_height)} ${wheel_offset_z}" rpy="${PI*0.5} 0 0"/>
+    </joint>
+    <joint name="joint_passive_wheel_r" type="fixed">
+        <parent link="vehicle_body"/>
+        <child link="passive_wheel_r"/>
+        <origin xyz="${0.5*body_x-wheel_radius} ${-0.5*(body_y+wheel_height)} ${wheel_offset_z}" rpy="${PI*0.5} 0 0"/>
     </joint>
     <!-- ==================track======================= -->
